File: hardware/NanoBud.brd (EAGLE design)
At the start: 50.8 x 43.1 mm, 8 parts

Commit message: dimension update
Other:
- board size 50.8 x 43.1 mm -> 50.9 x 43.2 mm
Changed lines of the file:
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@@
 <wire x1="19.05" y1="67.31" x2="15.24" y2="67.31" width="0.1524" layer="21"/>
 <text x="11.93" y="43.91" size="1.016" layer="21" rot="R90">GND</text>
-<wire x1="6.35" y1="63.5" x2="13.945" y2="71.095" width="0.1524" layer="21" curve="-100.388858"/>
-<wire x1="57.15" y1="35.56" x2="49.53" y2="27.94" width="0.1524" layer="21" curve="-90"/>
-<wire x1="48.235" y1="71.095" x2="57.15" y2="62.23" width="0.1524" layer="21" curve="-98.797411"/>
-<wire x1="15.24" y1="27.94" x2="6.35" y2="36.83" width="0.1524" layer="21" curve="-98.797411"/>
+<wire x1="6.35" y1="63.5" x2="13.945" y2="71.095" width="0.1524" layer="20" curve="-100.388858"/>
+<wire x1="57.15" y1="35.56" x2="49.53" y2="27.94" width="0.1524" layer="20" curve="-90"/>
+<wire x1="48.235" y1="71.095" x2="57.15" y2="62.23" width="0.1524" layer="20" curve="-98.797411"/>
+<wire x1="15.24" y1="27.94" x2="6.35" y2="36.83" width="0.1524" layer="20" curve="-98.797411"/>
 <wire x1="12.7" y1="58.42" x2="8.89" y2="58.42" width="0.1524" layer="21"/>
 <wire x1="8.89" y1="58.42" x2="8.89" y2="55.88" width="0.1524" layer="21"/>
